File: pcb/cad/ErgoDUE.kicad_sch (KiCad schematic)
At the start: 0 parts

Commit message: updated schematic information and produced pdf
Other:
- company: (none) -> Alessandro Rizzoni
Changed lines of the file:
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@@
     (date "2024-01-15")
     (rev "V0.1")
+    (company "Alessandro Rizzoni")
+    (comment 1 "SCHEMATIC")
+    (comment 2 "DRAFT")
+    (comment 3 "AIR")
   )
   (sheet (at 495.3 88.9) (size 38.1 25.4) (fields_autoplaced)

Commit message: wrapping up architecture
Changed lines of the file:
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@@
     (comment 2 "DRAFT")
     (comment 3 "AIR")
+    (comment 5 "ALL RESISTORS 1% 1/4W THIN FILM")
+    (comment 6 "ALL CAPACITORS 10% 1/4W X5R OR X7R DIELECTRIC")
+    (comment 7 "FOLLOW DATASHEET RECOMMENDATIONS FOR LAYOUT")
   )
-  (sheet (at 495.3 88.9) (size 38.1 25.4) (fields_autoplaced)
+  (sheet (at 495.3 12.7) (size 38.1 25.4) (fields_autoplaced)
     (stroke (width 0.1524) (type solid))
     (fill (color 0 0 0 0.0000))
-    (property "Sheetname" "USB Controller" (at 495.3 88.1884 0)
+    (property "Sheetname" "USB Controller" (at 495.3 11.9884 0)
       (effects (font (size 1.27 1.27)) (justify left bottom))
     )
-    (property "Sheetfile" "usbcontroller.kicad_sch" (at 495.3 114.8846 0)
-      (effects (font (size 1.27 1.27)) (justify left top))
-    )
-    (instances
-      (project "ErgoDUE"
-        (path "/4c935f39-219c-4006-ade5-f2ff1277cb0d" (page "11"))
-      )
-    )
-  )
-  (sheet (at 444.5 165.1) (size 38.1 25.4) (fields_autoplaced)
-    (stroke (width 0.1524) (type solid))
-    (fill (color 0 0 0 0.0000))
-    (property "Sheetname" "USB Downstream 1" (at 444.5 164.3884 0)
-      (effects (font (size 1.27 1.27)) (justify left bottom))
-    )
-    (property "Sheetfile" "downstream1.kicad_sch" (at 444.5 191.0846 0)
-      (effects (font (size 1.27 1.27)) (justify left top))
-    )
-    (instances
-      (project "ErgoDUE"
-        (path "/4c935f39-219c-4006-ade5-f2ff1277cb0d" (page "6"))
-      )
-    )
-  )
-  (sheet (at 444.5 50.8) (size 38.1 25.4) (fields_autoplaced)
-    (stroke (width 0.1524) (type solid))
-    (fill (color 0 0 0 0.0000))
-    (property "Sheetname" "Keyswitch Matrix" (at 444.5 50.0884 0)
-      (effects (font (size 1.27 1.27)) (justify left bottom))
-    )
-    (property "Sheetfile" "keyswitchmatrix.kicad_sch" (at 444.5 76.7846 0)
+    (property "Sheetfile" "usbcontroller.kicad_sch" (at 495.3 38.6846 0)
       (effects (font (size 1.27 1.27)) (justify left top))
     )
@@
       (project "ErgoDUE"
         (path "/4c935f39-219c-4006-ade5-f2ff1277cb0d" (page "3"))
+      )
+    )
+  )
+  (sheet (at 495.3 127) (size 38.1 25.4) (fields_autoplaced)
+    (stroke (width 0.1524) (type solid))
+    (fill (color 0 0 0 0.0000))
+    (property "Sheetname" "USB Downstream 1" (at 495.3 126.2884 0)
+      (effects (font (size 1.27 1.27)) (justify left bottom))
+    )
+    (property "Sheetfile" "downstream1.kicad_sch" (at 495.3 152.9846 0)
+      (effects (font (size 1.27 1.27)) (justify left top))
+    )
+    (instances
+      (project "ErgoDUE"
+        (path "/4c935f39-219c-4006-ade5-f2ff1277cb0d" (page "9"))
+      )
+    )
+  )
+  (sheet (at 495.3 50.8) (size 38.1 25.4) (fields_autoplaced)
+    (stroke (width 0.1524) (type solid))
+    (fill (color 0 0 0 0.0000))
+    (property "Sheetname" "Keyswitch Matrix" (at 495.3 50.0884 0)
+      (effects (font (size 1.27 1.27)) (justify left bottom))
+    )
+    (property "Sheetfile" "keyswitchmatrix.kicad_sch" (at 495.3 76.7846 0)
+      (effects (font (size 1.27 1.27)) (justify left top))
+    )
+    (instances
+      (project "ErgoDUE"
+        (path "/4c935f39-219c-4006-ade5-f2ff1277cb0d" (page "5"))
       )
     )
@@
     (instances
       (project "ErgoDUE"
-        (path "/4c935f39-219c-4006-ade5-f2ff1277cb0d" (page "4"))
+        (path "/4c935f39-219c-4006-ade5-f2ff1277cb0d" (page "6"))
       )
     )
   )
-  (sheet (at 444.5 241.3) (size 38.1 25.4) (fields_autoplaced)
+  (sheet (at 444.5 165.1) (size 38.1 25.4) (fields_autoplaced)
     (stroke (width 0.1524) (type solid))
     (fill (color 0 0 0 0.0000))
-    (property "Sheetname" "USB Downstream 3" (at 444.5 240.5884 0)
+    (property "Sheetname" "USB Downstream 3" (at 444.5 164.3884 0)
       (effects (font (size 1.27 1.27)) (justify left bottom))
     )
-    (property "Sheetfile" "downstream3.kicad_sch" (at 444.5 267.2846 0)
+    (property "Sheetfile" "downstream3.kicad_sch" (at 444.5 191.0846 0)
       (effects (font (size 1.27 1.27)) (justify left top))
     )
     (instances
       (project "ErgoDUE"
-        (path "/4c935f39-219c-4006-ade5-f2ff1277cb0d" (page "8"))
+        (path "/4c935f39-219c-4006-ade5-f2ff1277cb0d" (page "11"))
       )
     )
@@
     (instances
       (project "ErgoDUE"
-        (path "/4c935f39-219c-4006-ade5-f2ff1277cb0d" (page "5"))
+        (path "/4c935f39-219c-4006-ade5-f2ff1277cb0d" (page "8"))
       )
     )
   )
-  (sheet (at 495.3 50.8) (size 38.1 25.4) (fields_autoplaced)
+  (sheet (at 444.5 12.7) (size 38.1 25.4) (fields_autoplaced)
     (stroke (width 0.1524) (type solid))
     (fill (color 0 0 0 0.0000))
-    (property "Sheetname" "Microcontroller" (at 495.3 50.0884 0)
+    (property "Sheetname" "Microcontroller" (at 444.5 11.9884 0)
       (effects (font (size 1.27 1.27)) (justify left bottom))
     )
-    (property "Sheetfile" "microcontroller.kicad_sch" (at 495.3 76.7846 0)
+    (property "Sheetfile" "microcontroller.kicad_sch" (at 444.5 38.6846 0)
+      (effects (font (size 1.27 1.27)) (justify left top))
+    )
+    (instances
+      (project "ErgoDUE"
+        (path "/4c935f39-219c-4006-ade5-f2ff1277cb0d" (page "2"))
+      )
+    )
+  )
+  (sheet (at 495.3 88.9) (size 38.1 25.4) (fields_autoplaced)
+    (stroke (width 0.1524) (type solid))
+    (fill (color 0 0 0 0.0000))
+    (property "Sheetname" "LED Matrix" (at 495.3 88.1884 0)
+      (effects (font (size 1.27 1.27)) (justify left bottom))
+    )
+    (property "Sheetfile" "ledmatrix.kicad_sch" (at 495.3 114.8846 0)
+      (effects (font (size 1.27 1.27)) (justify left top))
+    )
+    (instances
+      (project "ErgoDUE"
+        (path "/4c935f39-219c-4006-ade5-f2ff1277cb0d" (page "7"))
+      )
+    )
+  )
+  (sheet (at 495.3 165.1) (size 38.1 25.4) (fields_autoplaced)
+    (stroke (width 0.1524) (type solid))
+    (fill (color 0 0 0 0.0000))
+    (property "Sheetname" "USB Downstream 2" (at 495.3 164.3884 0)
+      (effects (font (size 1.27 1.27)) (justify left bottom))
+    )
+    (property "Sheetfile" "downstream2.kicad_sch" (at 495.3 191.0846 0)
       (effects (font (size 1.27 1.27)) (justify left top))
     )
@@
     )
   )
-  (sheet (at 444.5 12.7) (size 38.1 25.4) (fields_autoplaced)
+  (sheet (at 444.5 50.8) (size 38.1 25.4) (fields_autoplaced)
     (stroke (width 0.1524) (type solid))
     (fill (color 0 0 0 0.0000))
-    (property "Sheetname" "LED Matrix" (at 444.5 11.9884 0)
+    (property "Sheetname" "Power" (at 444.5 50.0884 0)
       (effects (font (size 1.27 1.27)) (justify left bottom))
     )
-    (property "Sheetfile" "ledmatrix.kicad_sch" (at 444.5 38.6846 0)
+    (property "Sheetfile" "power.kicad_sch" (at 444.5 76.7846 0)
       (effects (font (size 1.27 1.27)) (justify left top))
     )
     (instances
       (project "ErgoDUE"
-        (path "/4c935f39-219c-4006-ade5-f2ff1277cb0d" (page "2"))
+        (path "/4c935f39-219c-4006-ade5-f2ff1277cb0d" (page "4"))
       )
     )
-  )
-  (sheet (at 444.5 203.2) (size 38.1 25.4) (fields_autoplaced)
-    (stroke (width 0.1524) (type solid))
-    (fill (color 0 0 0 0.0000))
-    (property "Sheetname" "USB Downstream 2" (at 444.5 202.4884 0)
-      (effects (font (size 1.27 1.27)) (justify left bottom))
-    )
-    (property "Sheetfile" "downstream2.kicad_sch" (at 444.5 229.1846 0)
-      (effects (font (size 1.27 1.27)) (justify left top))
-    )
-    (instances
-      (project "ErgoDUE"
-        (path "/4c935f39-219c-4006-ade5-f2ff1277cb0d" (page "7"))
-      )
-    )
-  )
-  (sheet (at 495.3 12.7) (size 38.1 25.4) (fields_autoplaced)
-    (stroke (width 0.1524) (type solid))
-    (fill (color 0 0 0 0.0000))
-    (property "Sheetname" "Power" (at 495.3 11.9884 0)
-      (effects (font (size 1.27 1.27)) (justify left bottom))
-    )
-    (property "Sheetfile" "power.kicad_sch" (at 495.3 38.6846 0)
-      (effects (font (size 1.27 1.27)) (justify left top))
-    )
-    (instances
-      (project "ErgoDUE"
-        (path "/4c935f39-219c-4006-ade5-f2ff1277cb0d" (page "9"))
-      )
-    )
