File: pcb/cad/downstream1.kicad_sch (KiCad schematic)
At the start: 14 parts, among them J601 USB_C_Receptacle, U601 ECMF02-2AMX6, U602 ECMF02-2AMX6, U603 ECMF02-2AMX6, U604 ECMF02-2AMX6, U605 ECMF02-2AMX6, U606 ECMF02-2AMX6, U607 CBTL02043A, U608 TUSB320, U609 PI3USB221E, U610 LM73100, U611 TPS25947xx

Commit message: moved old-old-old backups and finished preliminary USB architecture
Parts:
- removed U611: TPS25947xx, symbol Library:TI_TPS25947
- added C1: 7.5n, symbol Device:C
- added R10: 47k, symbol Device:R_US
- added R11: 17.8k, symbol Device:R_US
- added R2: 900k, symbol Device:R_US
- added R37, R6: 10k, symbol Device:R_US
- added R8: 150k, symbol Device:R_US
- added R9: 500k, symbol Device:R_US
Connections:
- net +5V: now also R9.1
- net GND: now also U610.9 (IMON), C1.2, R11.2, R8.2
- net I2C1_SCL: now also U608.8 (SCL/OUT2)
- net I2C1_SDA: now also U608.7 (SDA/OUT1)
- net ~{USB_DN1_DATA_EN}: now reaches U607.2 (XSD)
- net ~{USB_DN1_DATA_EN}: now also U608.11 (~{EN}), U609.6 (~{OE})
- net USB_DN1_RX+: now reaches U607.3 (A0_P)
- net USB_DN1_RX-: now reaches U607.4 (A0_N)
- net USB_DN1_TX+: now reaches U607.7 (A1_P)
- net USB_DN1_TX-: now reaches U607.8 (A1_N)
- net USB_DN1_POL: now reaches U607.9 (SEL)
- net USB_DN1_POL: now also U609.9 (SEL)
- net +3.3V: now reaches U608.12 (VDD)
- net +3.3V: now also R37.2, R6.1
- net at U608.3 (PORT): now also R37.1
- net at U608.4 (VBUS_DET): now also R2.2
- net at U608.5 (ADDR): now also R6.2
- net ~{USB_DN1_INT}: now reaches U608.6 (~{INT}/OUT3)
- net at J601.A4 (VBUS), J601.A9 (VBUS), J601.B4 (VBUS)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: now also R10.1, R2.1
- net USB_DN1_PWR_EN: now reaches U610.1 (EN/UVLO)
- net at U610.2 (OVLO): now also R8.1, R9.2
- net USB_DN1_PG: now reaches U610.3 (PG)
- net at U610.4 (PGTH): now also R10.2, R11.1
- net at U610.7 (DVDT): now also C1.1
- net USB_UP_DM renamed USB_DN1_DM
- net USB_UP_DP renamed USB_DN1_DP
- no-connect marks 8 -> 9
Other:
- moved on the sheet: U610

Commit message: updated schematic information and produced pdf
Other:
- company: (none) -> Alessandro Rizzoni
Changed lines of the file:
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@@
     (date "2024-01-15")
     (rev "V0.1")
+    (company "Alessandro Rizzoni")
+    (comment 1 "SCHEMATIC")
+    (comment 2 "DRAFT")
+    (comment 3 "AIR")
   )
   (junction (at 134.62 50.8) (diameter 0) (color 0 0 0 0)

Commit message: wrapping up architecture
Parts:
- renumbered C1 to C901, D601 to D901, D602 to D902, J601 to J901, R2 to R901, R37 to R902, R6 to R903, R10 to R904, R11 to R905, R9 to R906, R8 to R907, U601 to U901, U602 to U902, U603 to U903, U604 to U904, U605 to U905, U606 to U906, U607 to U907, U608 to U908, U609 to U909, U610 to U910

Commit message: usb architecture
Parts:
- removed R904: 47k, symbol Device:R_US
- removed R905: 17.8k, symbol Device:R_US
- removed R906: 500k, symbol Device:R_US
- removed R907: 150k, symbol Device:R_US
- removed U910: LM73100, symbol Library:TI_LM73100
- added C902, C903: C_Polarized_US, symbol Device:C_Polarized_US
- added C904: 100n, symbol Device:C
- added R908, R909, R910, R911, R912: R, symbol Device:R_US
- added U911: TPS25947x, symbol Library:TI_TPS25947
- C901: value 7.5n -> 100n
Connections:
- net +3V3: now also C901.1, C904.1
- net +5V: now also C902.1, R908.1, U911.5 (IN)
- net GND: now also U907.11 (GND), U907.20 (GND), U907.21 (GND), U907.5 (GND), C902.2, C903.2, C904.2, R910.2, R912.2, U911.8 (GND)
- net at J901.A4 (VBUS), J901.A9 (VBUS), J901.B4 (VBUS)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: now also C903.1, R911.1, U911.6 (OUT)
- new net: R911.2, R912.1, U911.4 (~{FLT}/PGTH)
- new net: R908.2, R909.1, U911.1 (EN/UVLO)
- new net: R909.2, R910.1, U911.2 (OVLO)
- new net USB_UP_PG: U911.3 (AUXOFF/PG)
Other:
- note added: "Take feedback from capacitor pad"
- moved on the sheet: U909

Commit message: ready for power circuitry
Parts:
- removed C904: 100n, symbol Device:C
- removed J901: USB_C_Receptacle, symbol Connector:USB_C_Receptacle
- removed U903, U904, U905, U906: ECMF02-2AMX6, Package_DFN_QFN:ST_UQFN-6L_1.5x1.7mm_P0.5mm, symbol Power_Protection:ECMF02-2AMX6
- removed U907: CBTL02043A, Package_DFN_QFN:WQFN-20-1EP_2.5x4.5mm_P0.5mm_EP1x2.9mm, symbol Analog_Switch:CBTL02043A
- added J901: USB_C_Receptacle_USB2.0_14P, symbol Connector:USB_C_Receptacle_USB2.0_14P
- renumbered C903 to C902, C902 to C903, R911 to R904, R912 to R905, R908 to R906, R909 to R907, R910 to R908, U908 to U903, U909 to U904, U911 to U905
Connections:
- net GND: now also J901.A1 (GND), J901.A12 (GND), J901.B1 (GND), J901.B12 (GND), J901.S1 (SHIELD)
- net at D902.1 (K), U903.1 (CC1): now also J901.A5 (CC1)
- net at D901.1 (K), U903.2 (CC2): now also J901.B5 (CC2)
- net at C902.1, R901.1, R904.1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: now also J901.A4 (VBUS), J901.A9 (VBUS), J901.B4 (VBUS), J901.B9 (VBUS)
- net at U902.1 (D+_in): now also J901.A6 (D+)
- net at U902.2 (D-_in): now also J901.B6 (D+)
- net at U901.1 (D+_in): now also J901.A7 (D-)
- net at U901.2 (D-_in): now also J901.B7 (D-)
- no-connect marks 9 -> 3
