File: pcb/cad/downstream2.kicad_sch (KiCad schematic)
At the start: 14 parts, among them J701 USB_C_Receptacle, U701 ECMF02-2AMX6, U702 ECMF02-2AMX6, U703 ECMF02-2AMX6, U704 ECMF02-2AMX6, U705 ECMF02-2AMX6, U706 ECMF02-2AMX6, U707 CBTL02043A, U708 TUSB320, U709 PI3USB221E, U710 LM73100, U711 TPS25947xx

Commit message: moved old-old-old backups and finished preliminary USB architecture
Parts:
- removed D701, D702: D_Zener_Filled, symbol Device:D_Zener_Filled
- removed J701: USB_C_Receptacle, symbol Connector:USB_C_Receptacle
- removed U701, U702, U703, U704, U705, U706: ECMF02-2AMX6, Package_DFN_QFN:ST_UQFN-6L_1.5x1.7mm_P0.5mm, symbol Power_Protection:ECMF02-2AMX6
- removed U707: CBTL02043A, Package_DFN_QFN:WQFN-20-1EP_2.5x4.5mm_P0.5mm_EP1x2.9mm, symbol Analog_Switch:CBTL02043A
- removed U708: TUSB320, Package_DFN_QFN:Texas_X2QFN-12_1.6x1.6mm_P0.4mm, symbol Interface_USB:TUSB320
- removed U709: PI3USB221E, symbol Library:DIODES_PI3USB221E
- removed U710: LM73100, symbol Library:TI_LM73100
- removed U711: TPS25947xx, symbol Library:TI_TPS25947
- added C3: 7.5n, symbol Device:C
- added D1, D2: D_Zener_Filled, symbol Device:D_Zener_Filled
- added J1: USB_C_Receptacle, symbol Connector:USB_C_Receptacle
- added R17: 900k, symbol Device:R_US
- added R18, R38: 10k, symbol Device:R_US
- added R19: 47k, symbol Device:R_US
- added R20: 17.8k, symbol Device:R_US
- added R31: 150k, symbol Device:R_US
- added R7: 500k, symbol Device:R_US
- added U1, U2, U3, U4, U5, U6: ECMF02-2AMX6, Package_DFN_QFN:ST_UQFN-6L_1.5x1.7mm_P0.5mm, symbol Power_Protection:ECMF02-2AMX6
- added U10: LM73100, symbol Library:TI_LM73100
- added U7: CBTL02043A, Package_DFN_QFN:WQFN-20-1EP_2.5x4.5mm_P0.5mm_EP1x2.9mm, symbol Analog_Switch:CBTL02043A
- added U8: TUSB320, Package_DFN_QFN:Texas_X2QFN-12_1.6x1.6mm_P0.4mm, symbol Interface_USB:TUSB320
- added U9: PI3USB221E, symbol Library:DIODES_PI3USB221E
Connections:
- net +3V3: now also U7.1 (VDD), U7.10 (VDD), U7.6 (VDD), U9.10 (VDD)
- net +5V: now also R7.1, U10.5 (IN)
- net GND: now also C3.2, D1.2 (A), D2.2 (A), R18.1, R20.2, R31.2, U1.3 (GND), U10.8 (GND), U10.9 (IMON), U2.3 (GND), U3.3 (GND), U4.3 (GND), U5.3 (GND), U6.3 (GND), U7.11 (GND), U7.20 (GND), U7.21 (GND), U7.5 (GND), U8.10 (GND), U9.5 (GND)
- net I2C1_SCL: now also U8.8 (SCL/OUT2)
- net I2C1_SDA: now also U8.7 (SDA/OUT1)
- new net: U6.5 (D-_out), U7.12 (C1_N)
- new net: U6.6 (D+_out), U7.13 (C1_P)
- new net: U5.5 (D-_out), U7.14 (C0_N)
- new net: U5.6 (D+_out), U7.15 (C0_P)
- new net: U4.5 (D-_out), U7.16 (B1_N)
- new net: U4.6 (D+_out), U7.17 (B1_P)
- new net: U3.5 (D-_out), U7.18 (B0_N)
- new net: U3.6 (D+_out), U7.19 (B0_P)
- new net: R38.1, U8.3 (PORT)
- new net: J1.B6 (D+), U2.1 (D+_in)
- new net: J1.B7 (D-), U2.2 (D-_in)
- new net: U2.5 (D-_out), U9.4 (2D-)
- new net: U2.6 (D+_out), U9.3 (2D+)
- new net: R18.2, U8.5 (ADDR)
- new net: D2.1 (K), J1.B5 (CC2), U8.1 (CC1)
- new net: D1.1 (K), J1.A5 (CC1), U8.2 (CC2)
- new net: R17.2, U8.4 (VBUS_DET)
- new net: C3.1, U10.7 (DVDT)
- new net: J1.A4 (VBUS), J1.A9 (VBUS), J1.B4 (VBUS), J1.B9 (VBUS), R17.1, R19.1, U10.6 (OUT)
- new net: J1.A6 (D+), U1.1 (D+_in)
- new net: J1.A7 (D-), U1.2 (D-_in)
- new net: U1.5 (D-_out), U9.2 (1D-)
- new net: U1.6 (D+_out), U9.1 (1D+)
- new net: R19.2, R20.1, U10.4 (PGTH)
- new net: J1.B3 (TX2-), U6.1 (D+_in)
- new net: J1.B2 (TX2+), U6.2 (D-_in)
- new net: R31.1, R7.2, U10.2 (OVLO)
- new net: J1.A1 (GND), J1.A12 (GND), J1.B1 (GND), J1.B12 (GND)
- new net: J1.A10 (RX2-), U5.1 (D+_in)
- new net: J1.A11 (RX2+), U5.2 (D-_in)
- new net: J1.A2 (TX1+), U4.2 (D-_in)
- new net: J1.A3 (TX1-), U4.1 (D+_in)
- new net: J1.B10 (RX1-), U3.1 (D+_in)
- new net: J1.B11 (RX1+), U3.2 (D-_in)
- new net +3.3V: R38.2, U8.12 (VDD)
- new net USB_DN2_DM: U9.7 (D-)
- new net USB_DN2_DP: U9.8 (D+)
- new net USB_DN2_PG: U10.3 (PG)
- new net USB_DN2_POL: U7.9 (SEL), U9.9 (SEL)
- new net USB_DN2_PWR_EN: U10.1 (EN/UVLO)
- new net USB_DN2_RX+: U7.3 (A0_P)
- new net USB_DN2_RX-: U7.4 (A0_N)
- new net USB_DN2_TX+: U7.7 (A1_P)
- new net USB_DN2_TX-: U7.8 (A1_N)
- new net ~{USB_DN2_DATA_EN}: U7.2 (XSD), U8.11 (~{EN}), U9.6 (~{OE})
- new net ~{USB_DN2_INT}: U8.6 (~{INT}/OUT3)
- no-connect marks 8 -> 9

Commit message: updated schematic information and produced pdf
Other:
- company: (none) -> Alessandro Rizzoni
Changed lines of the file:
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@@
     (date "2024-01-15")
     (rev "V0.1")
+    (company "Alessandro Rizzoni")
+    (comment 1 "SCHEMATIC")
+    (comment 2 "DRAFT")
+    (comment 3 "AIR")
   )
   (junction (at 377.19 80.01) (diameter 0) (color 0 0 0 0)

Commit message: wrapping up architecture
Parts:
- renumbered C3 to C1001, D1 to D1001, D2 to D1002, J1 to J1001, R17 to R1001, R38 to R1002, R18 to R1003, R19 to R1004, R20 to R1005, R7 to R1006, R31 to R1007, U1 to U1001, U2 to U1002, U3 to U1003, U4 to U1004, U5 to U1005, U6 to U1006, U7 to U1007, U8 to U1008, U9 to U1009, U10 to U1010

Commit message: usb architecture
Parts:
- added C1002, C1003: C_Polarized_US, symbol Device:C_Polarized_US
- added R1008, R1009, R1010, R1011, R1012: R, symbol Device:R_US
- added U1011: TPS25947x, symbol Library:TI_TPS25947
Connections:
- net GND: now also R1009.2, R1012.2
- net USB_DN2_PG: now also U1010.4 (PGTH); no longer U1010.3 (PG)
- net at R1004.2, R1005.1: now also U1010.3 (PG); no longer U1010.4 (PGTH)
- new net: R1010.2, R1011.1, U1011.1 (EN/UVLO)
- new net: R1011.2, R1012.1, U1011.2 (OVLO)
- new net: R1008.2, R1009.1, U1011.4 (~{FLT}/PGTH)
- new net: R1008.1, U1011.6 (OUT)
- new net: R1010.1, U1011.5 (IN)
- new net USB_UP_PG: U1011.3 (AUXOFF/PG)
Other:
- note added: "Take feedback from capacitor pad"

Commit message: ready for power circuitry
Parts:
- removed J1001: USB_C_Receptacle, symbol Connector:USB_C_Receptacle
- removed R1009, R1010, R1011, R1012: R, symbol Device:R_US
- removed U1003, U1004, U1005, U1006: ECMF02-2AMX6, Package_DFN_QFN:ST_UQFN-6L_1.5x1.7mm_P0.5mm, symbol Power_Protection:ECMF02-2AMX6
- removed U1007: CBTL02043A, Package_DFN_QFN:WQFN-20-1EP_2.5x4.5mm_P0.5mm_EP1x2.9mm, symbol Analog_Switch:CBTL02043A
- removed U1008: TUSB320, Package_DFN_QFN:Texas_X2QFN-12_1.6x1.6mm_P0.4mm, symbol Interface_USB:TUSB320
- removed U1009: PI3USB221E, symbol Library:DIODES_PI3USB221E
- removed U1010: LM73100, symbol Library:TI_LM73100
- removed U1011: TPS25947x, symbol Library:TI_TPS25947
- added J1001: USB_C_Receptacle_USB2.0_14P, symbol Connector:USB_C_Receptacle_USB2.0_14P
- added U1003: TUSB320, Package_DFN_QFN:Texas_X2QFN-12_1.6x1.6mm_P0.4mm, symbol Interface_USB:TUSB320
- added U1004: PI3USB221E, symbol Library:DIODES_PI3USB221E
- added U1005: TPS25947x, symbol Library:TI_TPS25947
- C1001: value 7.5n -> 100n
- R1004: value 47k -> R
- R1005: value 17.8k -> R
- R1006: value 500k -> R
- R1007: value 150k -> R
Connections:
- net +3.3V: now also R1003.1, U1003.12 (VDD)
- net +3V3: now also C1001.1, U1004.10 (VDD)
- net +5V: now also C1003.1, U1005.5 (IN)
- net GND: now also C1002.2, C1003.2, R1008.2, J1001.A1 (GND), J1001.A12 (GND), J1001.B1 (GND), J1001.B12 (GND), J1001.S1 (SHIELD), U1003.10 (GND), U1004.5 (GND), U1005.8 (GND); no longer R1003.1, R1007.2
- net I2C1_SCL: now also U1003.8 (SCL/OUT2)
- net I2C1_SDA: now also U1003.7 (SDA/OUT1)
- net USB_UP_PG: now also U1005.3 (AUXOFF/PG)
- net at R1002.1: now also U1003.3 (PORT)
- net at U1002.1 (D+_in): now also J1001.A6 (D+)
- net at U1002.2 (D-_in): now also J1001.B6 (D+)
- net at U1002.5 (D-_out): now also U1004.4 (2D-)
- net at U1002.6 (D+_out): now also U1004.3 (2D+)
- net at R1003.2: now also U1003.5 (ADDR)
- net at D1002.1 (K): now also J1001.A5 (CC1), U1003.1 (CC1)
- net at D1001.1 (K): now also J1001.B5 (CC2), U1003.2 (CC2)
- net at R1001.2: now also U1003.4 (VBUS_DET)
- net at R1008.1: now also R1007.2, U1005.2 (OVLO)
- net at R1001.1, R1004.1: now also C1002.1, J1001.A4 (VBUS), J1001.A9 (VBUS), J1001.B4 (VBUS), J1001.B9 (VBUS), U1005.6 (OUT)
- net at U1001.1 (D+_in): now also J1001.A7 (D-)
- net at U1001.2 (D-_in): now also J1001.B7 (D-)
- net at U1001.5 (D-_out): now also U1004.2 (1D-)
- net at U1001.6 (D+_out): now also U1004.1 (1D+)
- net at R1004.2, R1005.1: now also U1005.4 (~{FLT}/PGTH)
- net at R1006.2, R1007.1: now also U1005.1 (EN/UVLO)
- new net USB_DN1_DM: U1004.7 (D-)
- new net USB_DN1_DP: U1004.8 (D+)
- new net USB_DN1_POL: U1004.9 (SEL)
- new net ~{USB_DN1_DATA_EN}: U1003.11 (~{EN}), U1004.6 (~{OE})
- new net ~{USB_DN1_INT}: U1003.6 (~{INT}/OUT3)
- no-connect marks 9 -> 3
