File: pcb/cad/keyswitchmatrix.kicad_sch (KiCad schematic)
At the start: 93 parts, among them SW301 SW_Push, SW302 SW_Push, SW303 SW_Push, SW304 SW_Push, SW305 SW_Push, SW306 SW_Push, SW307 SW_Push, SW308 SW_Push, SW309 SW_Push, SW310 SW_Push, SW311 SW_Push, SW312 SW_Push, SW313 SW_Push, SW314 SW_Push, SW315 SW_Push, SW316 SW_Push, SW317 SW_Push, SW318 SW_Push, SW319 SW_Push, SW320 SW_Push, SW321 SW_Push, SW322 SW_Push, SW323 SW_Push, SW324 SW_Push, SW325 SW_Push, SW326 SW_Push, SW327 SW_Push, SW328 SW_Push, SW329 SW_Push, SW330 SW_Push, SW331 SW_Push, SW332 SW_Push, SW333 SW_Push, SW334 SW_Push, SW335 SW_Push, SW336 SW_Push, SW337 SW_Push, SW338 SW_Push, SW339 SW_Push, SW340 SW_Push, SW341 SW_Push, SW342 SW_Push, U301 MCP23017_ML

Commit message: updated schematic information and produced pdf
Other:
- company: (none) -> Alessandro Rizzoni
Changed lines of the file:
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@@
     (date "2024-01-15")
     (rev "V0.1")
+    (company "Alessandro Rizzoni")
+    (comment 1 "SCHEMATIC")
+    (comment 2 "DRAFT")
+    (comment 3 "AIR")
   )
   (junction (at 326.39 186.69) (diameter 0) (color 0 0 0 0)

Commit message: wrapping up architecture
Parts:
- renumbered C301 to C501, D301 to D501, D302 to D502, D303 to D503, D304 to D504, D305 to D505, D306 to D506, D307 to D507, D308 to D508, D309 to D509, D310 to D510, D311 to D511, D312 to D512, D313 to D513, D314 to D514, D315 to D515, D316 to D516, D317 to D517, D318 to D518, D319 to D519, D320 to D520, D321 to D521, D322 to D522, D323 to D523, D324 to D524, D325 to D525, D326 to D526, D327 to D527, D328 to D528, D329 to D529, D330 to D530, D331 to D531, D332 to D532, D333 to D533, D334 to D534, D335 to D535, D336 to D536, D337 to D537, D338 to D538, D339 to D539, D340 to D540, R301 to R501, R302 to R502, R303 to R503, R304 to R504, R305 to R505, R306 to R506, R307 to R507, R308 to R508, R309 to R509, SW301 to SW501, SW302 to SW502, SW303 to SW503, SW304 to SW504, SW305 to SW505, SW306 to SW506, SW307 to SW507, SW308 to SW508, SW309 to SW509, SW310 to SW510, SW311 to SW511, SW312 to SW512, SW313 to SW513, SW314 to SW514, SW315 to SW515, SW316 to SW516, SW317 to SW517, SW318 to SW518, SW319 to SW519, SW320 to SW520, SW321 to SW521, SW322 to SW522, SW323 to SW523, SW324 to SW524, SW325 to SW525, SW326 to SW526, SW327 to SW527, SW328 to SW528, SW329 to SW529, SW330 to SW530, SW331 to SW531, SW332 to SW532, SW333 to SW533, SW334 to SW534, SW335 to SW535, SW336 to SW536, SW337 to SW537, SW338 to SW538, SW339 to SW539, SW340 to SW540, SW341 to SW541, SW342 to SW542, U301 to U501

Commit message: usb architecture
Parts:
- C501: value C -> 100n
Changed lines of the file:
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@@
       (effects (font (size 1.27 1.27)) (justify left))
     )
-    (property "Value" "C" (at 139.7 110.49 0)
+    (property "Value" "100n" (at 139.7 110.49 0)
       (effects (font (size 1.27 1.27)) (justify left))
     )
