File: pcb/cad/leddrivers.kicad_sch (KiCad schematic)
At the start: 34 parts, among them U401 IS31FL3736, U402 IS31FL3736, U403 IS31FL3736

Commit message: updated schematic information and produced pdf
Other:
- company: (none) -> Alessandro Rizzoni
Changed lines of the file:
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@@
     (date "2024-01-15")
     (rev "V0.1")
+    (company "Alessandro Rizzoni")
+    (comment 1 "SCHEMATIC")
+    (comment 2 "DRAFT")
+    (comment 3 "AIR")
   )
   (junction (at 279.4 38.1) (diameter 0) (color 0 0 0 0)

Commit message: wrapping up architecture
Parts:
- renumbered C401 to C601, C402 to C602, C403 to C603, C404 to C604, C405 to C605, C406 to C606, C407 to C607, C408 to C608, C409 to C609, C410 to C610, C411 to C611, C412 to C612, C413 to C613, C414 to C614, C415 to C615, C416 to C616, C417 to C617, C418 to C618, C419 to C619, C420 to C620, C421 to C621, C422 to C622, C423 to C623, C424 to C624, R401 to R601, R402 to R602, R403 to R603, R404 to R604, R405 to R605, R406 to R606, R407 to R607, U401 to U601, U402 to U602, U403 to U603

Commit message: usb architecture
Parts:
- C601, C602, C603, C604, C605, C606, C607, C608, C617, C618, C619, C620: value C -> 1u
- C609, C610, C611, C612, C613, C614, C615, C616, C621, C622, C623, C624: value C -> 100n

Commit message: ready for power circuitry
Parts:
- renumbered C605 to C601, C617 to C602, C618 to C604, C601 to C605, C619 to C606, C620 to C608, C613 to C609, C621 to C610, C622 to C612, C609 to C613, C623 to C614, C624 to C616, C602 to C617, C604 to C618, C606 to C619, C608 to C620, C610 to C621, C612 to C622, C614 to C623, C616 to C624
