File: pcb/cad/ledmatrix.kicad_sch (KiCad schematic)
At the start: 52 parts

Commit message: updated schematic information and produced pdf
Other:
- company: (none) -> Alessandro Rizzoni
Changed lines of the file:
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@@
     (date "2024-01-15")
     (rev "V0.1")
+    (company "Alessandro Rizzoni")
+    (comment 1 "SCHEMATIC")
+    (comment 2 "DRAFT")
+    (comment 3 "AIR")
   )
   (junction (at 52.07 92.71) (diameter 0) (color 0 0 0 0)

Commit message: wrapping up architecture
Parts:
- renumbered D201 to D701, D202 to D702, D203 to D703, D204 to D704, D205 to D705, D206 to D706, D207 to D707, D208 to D708, D209 to D709, D210 to D710, D211 to D711, D212 to D712, D213 to D713, D214 to D714, D215 to D715, D216 to D716, D217 to D717, D218 to D718, D219 to D719, D220 to D720, D221 to D721, D222 to D722, D223 to D723, D224 to D724, D225 to D725, D226 to D726, D227 to D727, D228 to D728, D229 to D729, D230 to D730, D231 to D731, D232 to D732, D233 to D733, D234 to D734, D235 to D735, D236 to D736, D237 to D737, D238 to D738, D239 to D739, D240 to D740, D241 to D741, D242 to D742, D243 to D743, D244 to D744, D245 to D745, D246 to D746, D247 to D747, D248 to D748, D249 to D749, D250 to D750, D251 to D751, D252 to D752
