File: pcb/cad/microcontroller.kicad_sch (KiCad schematic)
At the start: 29 parts, among them J1001 Conn_01x04_Pin, SW1001 SW_Push, SW1002 SW_Push, U1001 AT25xxx-MA, U1002 RP2040, Y1001 Crystal_GND24

Commit message: moved old-old-old backups and finished preliminary USB architecture
Connections:
- net ~{USB_DN1_INT}: now reaches U1002.15 (GPIO12)
- net USB_DN1_POL: now reaches U1002.16 (GPIO13)
- net USB_DN1_PWR_EN: now reaches U1002.17 (GPIO14)
- net USB_DN1_DATA_EN: now reaches U1002.18 (GPIO15)
- net ~{USB_DN2_INT}: now reaches U1002.27 (GPIO16)
- net USB_DN2_POL: now reaches U1002.28 (GPIO17)
- net USB_DN2_PWR_EN: now reaches U1002.29 (GPIO18)
- net USB_DN2_PWR_EN: now also U1002.34 (GPIO22)
- net USB_DN2_DATA_EN: now reaches U1002.30 (GPIO19)
- net USB_DN2_DATA_EN: now also U1002.35 (GPIO23)
- net ~{USB_DN3_INT}: now reaches U1002.31 (GPIO20)
- net USB_DN3_POL: now reaches U1002.32 (GPIO21)
Other:
- note added: "1MHz I2C to: GPIO Expander LED Drivers USB Port Controller 3"
- note added: "1MHz I2C to: USB Hub Controller USB Port Controllers 1 and 2"
- note removed: "1MHz I2C to: GPIO Expander LED Drivers"
- note removed: "1MHz I2C to: USB Hub Controller USB Port Controllers"
- moved on the sheet: D1001, J1001

Commit message: updated schematic information and produced pdf
Other:
- company: (none) -> Alessandro Rizzoni
Changed lines of the file:
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@@
     (date "2024-01-15")
     (rev "V0.1")
+    (company "Alessandro Rizzoni")
+    (comment 1 "SCHEMATIC")
+    (comment 2 "DRAFT")
+    (comment 3 "AIR")
   )
   (junction (at 273.05 113.03) (diameter 0) (color 0 0 0 0)

Commit message: wrapping up architecture
Parts:
- renumbered C1001 to C201, C1002 to C202, C1003 to C203, C1004 to C204, C1005 to C205, C1006 to C206, C1007 to C207, C1008 to C208, C1009 to C209, C1010 to C210, C1011 to C211, D1001 to D201, D1002 to D202, J1001 to J201, R1001 to R201, R1002 to R202, R1003 to R203, R1004 to R204, R1005 to R205, R1006 to R206, R1007 to R207, R1008 to R208, R1009 to R209, R1010 to R210, SW1001 to SW201, SW1002 to SW202, U1001 to U201, U1002 to U202, Y1001 to Y201
Connections:
- net USB_GLBL_RST: now reaches U202.36 (GPIO24)
- net USB_UP_PG: now reaches U202.38 (GPIO26_ADC0)
- net USB_DN1_PG: now reaches U202.39 (GPIO27_ADC1)
- net USB_DN2_PG: now reaches U202.40 (GPIO28_ADC2)
- net USB_DN3_PG: now reaches U202.41 (GPIO29_ADC3)
