File: pcb/cad/power.kicad_sch (KiCad schematic)
At the start: 16 parts, among them U901 AP3401, U902 AP3401

Commit message: updated schematic information and produced pdf
Other:
- company: (none) -> Alessandro Rizzoni
Changed lines of the file:
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@@
     (date "2024-01-15")
     (rev "V0.1")
+    (company "Alessandro Rizzoni")
+    (comment 1 "SCHEMATIC")
+    (comment 2 "DRAFT")
+    (comment 3 "AIR")
   )
   (junction (at 167.64 85.09) (diameter 0) (color 0 0 0 0)

Commit message: wrapping up architecture
Parts:
- renumbered C901 to C401, C902 to C402, C903 to C403, C904 to C404, L901 to L401, L902 to L402, R901 to R401, R902 to R402, R903 to R403, R904 to R404, R905 to R405, R906 to R406, R907 to R407, R908 to R408, U901 to U401, U902 to U402
