File: pcb/cad/upstream.kicad_sch (KiCad schematic)
At the start: 12 parts, among them J501 USB_C_Receptacle, U501 LM73100, U502 TPS25947xx, U503 ECMF02-2AMX6, U504 ECMF02-2AMX6, U505 ECMF02-2AMX6, U506 ECMF02-2AMX6, U507 ECMF02-2AMX6, U508 ECMF02-2AMX6, U509 CYPD3177-24LQ, U510 PI3USB221E, U511 CBTL02043A

Commit message: moved old-old-old backups and finished preliminary USB architecture
Parts:
- removed U502: TPS25947xx, symbol Library:TI_TPS25947
- removed U509: CYPD3177-24LQ, Package_DFN_QFN:QFN-24-1EP_4x4mm_P0.5mm_EP2.75x2.75mm, symbol Interface_USB:CYPD3177-24LQ
- added C2: 7.5n, symbol Device:C
- added R12: 47k, symbol Device:R_US
- added R13: 17.8k, symbol Device:R_US
- added R14: 470k, symbol Device:R_US
- added R15: 33.2k, symbol Device:R_US
- added R16: 147k, symbol Device:R_US
- added R35: 10k, symbol Device:R_US
- added R36: 900k, symbol Device:R_US
- added U21: TUSB320, Package_DFN_QFN:Texas_X2QFN-12_1.6x1.6mm_P0.4mm, symbol Interface_USB:TUSB320
Connections:
- net GND: now also U501.9 (IMON), U510.6 (~{OE}), U511.2 (XSD), C2.2, R13.2, R16.2, R35.1, U21.10 (GND), U21.11 (~{EN}), U21.3 (PORT)
- net at U501.1 (EN/UVLO): now also R14.2, R15.1
- net at U501.2 (OVLO): now also R15.2, R16.1
- net USB_DN1_PG: now reaches U501.3 (PG)
- net at U501.4 (PGTH): now also R12.2, R13.1
- net at U501.5 (IN): now also J501.A4 (VBUS), J501.A9 (VBUS), J501.B4 (VBUS), J501.B9 (VBUS), R14.1, R36.1
- net +5V: now reaches U501.6 (OUT)
- net +5V: now also R12.1
- net at U501.7 (DVDT): now also C2.1
- net at J501.A5 (CC1): now also U21.2 (CC2)
- net at J501.B5 (CC2): now also U21.1 (CC1)
- net USB_UP_POL: now reaches U511.9 (SEL)
- net USB_UP_POL: now also U510.9 (SEL)
- new net: R35.2, U21.5 (ADDR)
- new net: R36.2, U21.4 (VBUS_DET)
- new net +3.3V: U21.12 (VDD)
- new net I2C0_SCL: U21.8 (SCL/OUT2)
- new net I2C0_SDA: U21.7 (SDA/OUT1)
- new net ~{USB_UP_INT}: U21.6 (~{INT}/OUT3)
- no-connect marks 8 -> 9
Other:
- moved on the sheet: U501

Commit message: updated schematic information and produced pdf
Other:
- company: (none) -> Alessandro Rizzoni
Changed lines of the file:
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@@
     (date "2024-01-15")
     (rev "V0.1")
+    (company "Alessandro Rizzoni")
+    (comment 1 "SCHEMATIC")
+    (comment 2 "DRAFT")
+    (comment 3 "AIR")
   )
   (junction (at 273.05 71.12) (diameter 0) (color 0 0 0 0)

Commit message: wrapping up architecture
Parts:
- renumbered C2 to C801, J501 to J801, R36 to R801, R35 to R802, R14 to R803, R15 to R804, R16 to R805, R12 to R806, R13 to R807, U503 to U801, U504 to U802, U505 to U803, U506 to U804, U507 to U805, U508 to U806, U511 to U807, U21 to U808, U510 to U809, U501 to U810
Connections:
- net USB_DN1_PG renamed USB_UP_PG

Commit message: usb architecture
Parts:
- removed C801: 7.5n, symbol Device:C
- removed U810: LM73100, symbol Library:TI_LM73100
- added C802, C803, C804: C, symbol Device:C
- added C805, C806: C_Polarized_US, symbol Device:C_Polarized_US
- added U811: TPS25947x, symbol Library:TI_TPS25947
- R803: value 470k -> R
- R804: value 33.2k -> R
- R805: value 147k -> R
- R806: value 47k -> R
- R807: value 17.8k -> R
Connections:
- net +5V: now also U811.6 (OUT)
- net USB_UP_PG: now also U811.3 (AUXOFF/PG)
- net at R803.2, R804.1: now also U811.1 (EN/UVLO)
- net at R804.2, R805.1: now also U811.2 (OVLO)
- net at R806.2, R807.1: now also U811.4 (~{FLT}/PGTH)
- net at J801.A4 (VBUS), J801.A9 (VBUS), J801.B4 (VBUS)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: now also U811.5 (IN)
Other:
- note added: "Take feedback from capacitor pad"

Commit message: starting to clean up for usb2.0
Parts:
- removed C802, C804: C, symbol Device:C
- removed J801: USB_C_Receptacle, symbol Connector:USB_C_Receptacle
- removed U803, U804, U805, U806: ECMF02-2AMX6, Package_DFN_QFN:ST_UQFN-6L_1.5x1.7mm_P0.5mm, symbol Power_Protection:ECMF02-2AMX6
- removed U807: CBTL02043A, Package_DFN_QFN:WQFN-20-1EP_2.5x4.5mm_P0.5mm_EP1x2.9mm, symbol Analog_Switch:CBTL02043A
- added C801: 100n, symbol Device:C
- added J802: USB_C_Receptacle_USB2.0_14P, symbol Connector:USB_C_Receptacle_USB2.0_14P
- C803: value C -> 100n
Connections:
- net +3.3V: now also C801.1
- net +3V3: now also C803.1
- net GND: now also C803.2, C801.2, J802.A1 (GND), J802.A12 (GND), J802.B1 (GND), J802.B12 (GND), J802.S1 (SHIELD)
- net at U801.1 (D+_in): now also J802.A7 (D-)
- net at U801.2 (D-_in): now also J802.B7 (D-)
- net at R801.1, R803.1, U811.5 (IN): now also J802.A4 (VBUS), J802.A9 (VBUS), J802.B4 (VBUS), J802.B9 (VBUS)
- net at U802.1 (D+_in): now also J802.A6 (D+)
- net at U802.2 (D-_in): now also J802.B6 (D+)
- net at U808.2 (CC2): now also J802.B5 (CC2)
- net at U808.1 (CC1): now also J802.A5 (CC1)
- no-connect marks 9 -> 3
Other:
- moved on the sheet: C803, U801, U809

Commit message: ready for power circuitry
Parts:
- renumbered C803 to C801, C801 to C802, C805 to C803, C806 to C804, J802 to J801, U808 to U803, U809 to U804, U811 to U805
