File: pcb/cad/usbcontroller.kicad_sch (KiCad schematic)
At the start: 17 parts, among them U11001 TUSB8041, Y11001 Crystal_GND24

Commit message: moved old-old-old backups and finished preliminary USB architecture
Parts:
- added R1, R27, R28, R29, R30, R33: 10k, symbol Device:R_US
- added R3, R4, R5: 4.7k, symbol Device:R_US
- added R32: 9.53k, symbol Device:R_US
- added R34: 90.9k, symbol Device:R_US
Connections:
- net GND: now also U11001.65 (VSS), R29.1, R30.1, R32.1, R33.1
- net uC_USB_DM: now also U11001.25 (USB_DM_DN4); no longer U11001.2 (USB_DM_DN1)
- net uC_USB_DP: now also U11001.24 (USB_DP_DN4); no longer U11001.1 (USB_DP_DN1)
- net at C11001.1, C11003.1, C11004.1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: now also C11002.1, U11001.16 (VDD33), U11001.34 (VDD33), U11001.52 (VDD33), U11001.63 (VDD33)
- net at C11007.1, C11009.1, C11011.1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: now also C11005.1, C11008.1, C11010.1, C11012.1, C11014.1, U11001.13 (VDD), U11001.21 (VDD), U11001.28 (VDD), U11001.31 (VDD), U11001.5 (VDD), U11001.51 (VDD), U11001.57 (VDD), U11001.8 (VDD)
- net USB_DN2_DM: now reaches U11001.10 (USB_DM_DN2)
- net USB_DN2_TX+: now reaches U11001.11 (USB_SSTXP_DN2)
- net USB_DN2_TX-: now reaches U11001.12 (USB_SSTXM_DN2)
- net USB_DN2_RX+: now reaches U11001.14 (USB_SSRXP_DN2)
- net USB_DN2_RX-: now reaches U11001.15 (USB_SSRXM_DN2)
- net USB_DN3_DP: now reaches U11001.17 (USB_DP_DN3)
- net USB_DN3_DM: now reaches U11001.18 (USB_DM_DN3)
- net USB_DN3_TX+: now reaches U11001.19 (USB_SSTXP_DN3)
- net USB_DN3_TX-: now reaches U11001.20 (USB_SSTXM_DN3)
- net USB_DN3_RX+: now reaches U11001.22 (USB_SSRXP_DN3)
- net USB_DN3_RX-: now reaches U11001.23 (USB_SSRXM_DN3)
- net USB_DN1_TX+: now reaches U11001.3 (USB_SSTXP_DN1)
- net at U11001.33 (PWRCTL3/BATEN3): now also R5.1
- net at U11001.35 (PWRCTL2/BATEN2): now also R4.1
- net at U11001.36 (PWRCTL1/BATEN1): now also R3.1
- net at U11001.39 (SMBUSz/SS_SUSPEND): now also R1.1
- net USB_DN1_TX-: now reaches U11001.4 (USB_SSTXM_DN1)
- net at U11001.40 (FULLPWRMGMTz/SMBA1/SS_UP): now also R29.2
- net at U11001.41 (PWRCTL_POL): now also R27.1
- net at U11001.42 (GANGED/SMBA2/HS_UP): now also R30.2
- net at U11001.45 (AUTOENz/HS_SUSPEND): now also R28.1
- net at U11001.48 (USB_VBUS): now also R33.2, R34.1
- net USB_GLBL_RST: now reaches U11001.50 (GRSTz)
- net USB_DN1_RX+: now reaches U11001.6 (USB_SSRXP_DN1)
- net at U11001.64 (USB_R1): now also R32.2
- net USB_DN1_RX-: now reaches U11001.7 (USB_SSRXM_DN1)
- net USB_DN2_DP: now reaches U11001.9 (USB_DP_DN2)
- new net +3.3V: R1.2, R27.2, R28.2, R3.2, R4.2, R5.2
- new net +5V: R34.2
- new net USB_DN1_DM: U11001.2 (USB_DM_DN1)
- new net USB_DN1_DP: U11001.1 (USB_DP_DN1)
- no-connect marks 0 -> 11
Other:
- note added: "Look closer at bettery charging..."
- moved on the sheet: C11001, C11002, C11003, C11004, C11005, C11006, C11007, C11008, C11009, C11010, C11011, C11012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

Commit message: updated schematic information and produced pdf
Other:
- company: (none) -> Alessandro Rizzoni
Changed lines of the file:
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@@
     (date "2024-01-15")
     (rev "V0.1")
+    (company "Alessandro Rizzoni")
+    (comment 1 "SCHEMATIC")
+    (comment 2 "DRAFT")
+    (comment 3 "AIR")
   )
   (junction (at 316.23 90.17) (diameter 0) (color 0 0 0 0)

Commit message: wrapping up architecture
Parts:
- renumbered C11001 to C301, C11003 to C302, C11004 to C303, C11006 to C304, C11002 to C305, C11005 to C306, C11007 to C307, C11009 to C308, C11011 to C309, C11013 to C310, C11008 to C311, C11010 to C312, C11012 to C313, C11014 to C314, R28 to R301, R29 to R302, R27 to R303, R30 to R304, R11001 to R305, R34 to R306, R33 to R307, R1 to R308, R32 to R309, R3 to R310, R4 to R311, R5 to R312, U11001 to U301, Y11001 to Y301

Commit message: starting to clean up for usb2.0
Parts:
- removed C314: 100n, symbol Device:C
- removed U301: TUSB8041, Package_DFN_QFN:QFN-64-1EP_9x9mm_P0.5mm_EP6x6mm_ThermalVias, symbol Interface_USB:TUSB8041
- added U301: TUSB4041I, Package_QFP:HTQFP-64-1EP_10x10mm_P0.5mm_EP8x8mm_Mask4.4x4.4mm_ThermalVias, symbol Interface_USB:TUSB4041I
Connections:
- net GND: now also U301.65 (VSS)
- net I2C1_SCL: now also U301.6 (SCL/SMBCLK)
- net I2C1_SDA: now also U301.5 (SDA/SMBDAT)
- net USB_DN1_DM: now also U301.34 (USB_DM_DN1)
- net USB_DN1_DP: now also U301.33 (USB_DP_DN1)
- net USB_DN2_DM: now also U301.42 (USB_DM_DN2)
- net USB_DN2_DP: now also U301.41 (USB_DP_DN2)
- net USB_DN3_DM: now also U301.50 (USB_DM_DN3)
- net USB_DN3_DP: now also U301.49 (USB_DP_DN3)
- net USB_GLBL_RST: now also U301.18 (GRSTz)
- net USB_UP_DM: now also U301.22 (USB_DM_UP)
- net USB_UP_DP: now also U301.21 (USB_DP_UP)
- net uC_USB_DM: now also U301.57 (USB_DM_DN4)
- net uC_USB_DP: now also U301.56 (USB_DP_DN4)
- net at C301.1, C302.1, C303.1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: now also U301.2 (VDD33), U301.20 (VDD33), U301.31 (VDD33), U301.48 (VDD33)
- net at C306.1, C307.1, C308.1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: now also U301.19 (VDD), U301.25 (VDD), U301.37 (VDD), U301.45 (VDD), U301.53 (VDD), U301.60 (VDD), U301.63 (VDD)
- net at R310.1: now also U301.4 (PWRCTL1/BATEN1)
- net at R302.2: now also U301.10 (GANGED/SMBA2/HS_UP)
- net at R303.1: now also U301.8 (FULLPWRMGMTz/SMBA1)
- net at R309.2: now also U301.32 (USB_R1)
- net at R306.1, R307.2: now also U301.16 (USB_VBUS)
- net at R305.2: now also U301.29 (XO)
- net at Y301.3: now also U301.30 (XI)
- net at R301.1: now also U301.9 (PWRCTL_POL)
- net at R304.2: now also U301.13 (AUTOENz/HS_SUSPEND)
- net at R311.1: now also U301.3 (PWRCTL2/BATEN2)
- net at R312.1: now also U301.1 (PWRCTL3/BATEN3)
- net at R308.1: now also U301.7 (SMBUSz)
- no-connect marks 11 -> 6
Other:
- moved on the sheet: R309
